File: uav_pcb_1.kicad_sch (KiCad schematic)
At the start: 28 parts, among them J1 Conn_01x02_Pin, J2 Conn_02x08_Odd_Even, U1 STM32F405RGTx, U2 MPU-6050, U3 BMP280, U4 LIS3MDL, U5 PCA9685BS

Commit message: Add schematic file 2 via upload
Parts:
- removed D1: GRN, symbol Device:LED
- removed D2: RED, symbol Device:LED
- removed D3: YLW, symbol Device:LED
- removed D4: BLU, symbol Device:LED
- removed J1: Conn_01x02_Pin, symbol Connector:Conn_01x02_Pin
- removed R1, R2, R3, R4: 1k, symbol Device:R
- removed U2: MPU-6050, Sensor_Motion:InvenSense_QFN-24_4x4mm_P0.5mm, symbol Sensor_Motion:MPU-6050
- removed U3: BMP280, Package_LGA:Bosch_LGA-8_2x2.5mm_P0.65mm_ClockwisePinNumbering, symbol Sensor_Pressure:BMP280
- removed U4: LIS3MDL, Package_LGA:LGA-12_2x2mm_P0.5mm, symbol Sensor_Magnetic:LIS3MDL
- added C22, C25, C26, C27, C30: 100n, symbol Device:C
- added C23, C24: 10u, symbol Device:C
- added C29: 1u, symbol Device:C
- added C31, C32: 10p, symbol Device:C
- added D6: GR, symbol Device:LED
- added D7: D_Schottky, symbol Device:D_Schottky
- added F1: Fuse, symbol Device:Fuse
- added FB1, FB2: FerriteBead_Small, symbol Device:FerriteBead_Small
- added J1: USB_B_Micro, symbol Connector:USB_B_Micro
- added R12, R13, R14, R15, R16: R, symbol Device:R
- added R7: 1k, symbol Device:R
- added R8, R9: 22, symbol Device:R
- added U10: CH330N, Package_SO:SOIC-8_3.9x4.9mm_P1.27mm, symbol Interface_USB:CH330N
- added U4: SN74LVC1G04DCKR, SN74LVC1G04DCKR:SOT65P210X110-5N, symbol SN74LVC1G04DCKR:SN74LVC1G04DCKR
- added U8: LD39200PU33R, LD39200PU33R:SON95P300X300X100-7N, symbol LD39200PU33R:LD39200PU33R
- added U9: USBLC6-2SC6, Package_TO_SOT_SMD:SOT-23-6, symbol Power_Protection:USBLC6-2SC6
- added Y1: Crystal_GND24, symbol Device:Crystal_GND24
Connections:
- net 12C1_SCL: no longer U1.39 (PC8)
- net 12C1_SDA: no longer U1.62 (PB9)
- net GND: now also C22.2, C23.2, C24.2, C25.1, C26.1, C27.2, C29.2, C30.2, C31.2, C32.2, J1.5 (GND), J1.6 (Shield), R7.2, U10.3 (GND), U4.3 (GND), U8.3 (GND), U8.7 (EXP), U9.2 (GND), Y1.2, Y1.4
- net BAR_CSB: no longer names the net of U1.28 (PB2)
- net BAR_SCK: no longer names the net of U1.26 (PB0)
- net BAR_SDI: no longer names the net of U1.27 (PB1)
- net IMU_SCL: no longer names the net of U1.15 (PA1)
- net IMU_SDA: no longer names the net of U1.14 (PA0)
- net LED_A: no longer names the net of U1.33 (PB12)
- net LED_B: no longer names the net of U1.34 (PB13)
- net LED_C: no longer names the net of U1.35 (PB14)
- net LED_D: no longer names the net of U1.36 (PB15)
- net MAG_C1: no longer names the net of U1.24 (PC4)
- net MAG_CS: no longer names the net of U1.8 (PC0)
- net MAG_SCL: no longer names the net of U1.9 (PC1)
- net MAG_SDA: no longer names the net of U1.10 (PC2)
- net MAG_SDO: no longer names the net of U1.11 (PC3)
- new net: D6.1 (K), R7.1
- new net: C27.1, D7.2 (A), FB1.2, U9.5 (VBUS)
- new net: R9.1, U10.7 (RXD)
- new net: F1.2, FB1.1
- new net: C32.1, R16.1, Y1.3
- new net: R8.1, U10.6 (TXD)
- new net: C25.2, U10.8 (V3)
- new net: F1.1, J1.1 (VBUS)
- new net +3V3: C22.1, C23.1, C24.1, C26.2, D6.2 (A), D7.1 (K), FB2.2, R12.1, R13.1, R14.1, R15.1, U10.5 (VCC), U4.5 (VCC), U8.1 (OUT), U8.2 (SENSE), U8.5 (EN), U8.6 (IN)
- new net HSE_IN: C31.1, Y1.1
- new net HSE_OUT: R16.2
- new net I2C1_SCL: R12.2
- new net I2C1_SDA: R13.2
- new net I2C3_SCL: R14.2
- new net I2C3_SDA: R15.2
- new net UART3_RX: R9.2
- new net UART3_TX: R8.2
- new net UART4_RX: U4.4 (Y)
- new net UART4_RX_INV: U4.2 (A)
- new net USB_CONN_D+: J1.3 (D+), U9.6 (I/O1)
- new net USB_CONN_D-: J1.2 (D-), U10.2 (UD-), U9.4 (I/O2)
- new net USB_CONV_D+: U10.1 (UD+), U9.1 (I/O1)
- new net USB_CONV_D-: U9.3 (I/O2)
- new net VDDA: C29.1, C30.1, FB2.1
- no-connect marks 24 -> 12
Other:
- added sheet sensors (untitled.kicad_sch)
- moved on the sheet: C10, C11, C2, C3, C4, C5, C6, C7, C8, C9, D5, J2

Commit message: Add files via upload
Parts:
- added C33, C34: C, symbol Device:C
- added R17: 0R, symbol Device:R
- Y1: value Crystal_GND24 -> 25MHz
Connections:
- net +3V3: now also D5.1 (K), U1.1 (VBAT), U1.19 (VDD), U1.32 (VDD), U1.48 (VDD), U1.64 (VDD)
- net GND: now also U1.12 (VSSA), U1.18 (VSS), U1.63 (VSS), C33.2, C34.2
- net HSE_IN: now also U1.5 (PH0)
- net HSE_OUT: now also U1.6 (PH1)
- net I2C1_SCL: now also U1.61 (PB8)
- net I2C1_SDA: now also U1.62 (PB9)
- net I2C3_SCL: now also U1.41 (PA8)
- net I2C3_SDA: now also U1.40 (PC9)
- net UART3_RX: now also U1.52 (PC11)
- net UART3_TX: now also U1.51 (PC10)
- net UART4_RX: now also U1.15 (PA1)
- net INT_MAG: now reaches U1.10 (PC2)
- net INT_BAR: now reaches U1.11 (PC3)
- net UART4_TX: now reaches U1.14 (PA0)
- net UART2_TX: now reaches U1.16 (PA2)
- net UART2_RX: now reaches U1.17 (PA3)
- net SPI1_SCK: now reaches U1.21 (PA5)
- net SPI1_MISO: now reaches U1.22 (PA6)
- net SPI1_MOSI: now reaches U1.23 (PA7)
- net SPI1_CS: now reaches U1.24 (PC4)
- net FLASH_!WP: now reaches U1.25 (PC5)
- net BOOT1: now reaches U1.28 (PB2)
- net TIM2_CH3: now reaches U1.29 (PB10)
- net TIM2_CH4: now reaches U1.30 (PB11)
- net at U1.31 (VCAP_1): now also C33.1
- net LED_A: now reaches U1.33 (PB12)
- net LED_B: now reaches U1.34 (PB13)
- net LED_C: now reaches U1.35 (PB14)
- net LED_D: now reaches U1.36 (PB15)
- net SWDIO: now reaches U1.46 (PA13)
- net at U1.47 (VCAP_2): now also C34.1
- net SWCLK: now reaches U1.49 (PA14)
- net TIM2_CH1: now reaches U1.50 (PA15)
- net TIM2_CH2: now reaches U1.55 (PB3)
- net UART1_TX: now reaches U1.58 (PB6)
- net UART1_RX: now reaches U1.59 (PB7)
- net BOOT0: now reaches U1.60 (BOOT0)
- net NRST: now reaches U1.7 (NRST)
- net INT_ACC: now reaches U1.8 (PC0)
- net INT_GYR: now reaches U1.9 (PC1)
- net at J2.1 (Pin_1), J2.11 (Pin_11), J2.13 (Pin_13)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: now also R17.1
- net at D5.2 (A): now also R17.2
- no-connect marks 12 -> 29
Other:
- note added: "Decoupling Capacitors"
- note added: "High-Speed External Crystal"
- note added: "I2C Pull-Ups"
- note added: "PWM DRIVER"
- note added: "PWM_PWR1 Conn_02x08_Odd_Even"
- note added: "Power"
- note added: "SBUS Inverter"
- note added: "USB"
- moved on the sheet: C1, C10, C11, C2, C22, C23, C24, C25, C26, C27, C29, C3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
